File: kicad/keyboard.kicad_pcb (KiCad board)
At the start: 2 copper layers, 297.2 x 104.8 mm, 86 parts, among them J1 Conn_01x11_Female, J2 Conn_01x03_Male, SW1 SW_Push, SW10 Gateron_ks_27, SW11 Gateron_ks_27, SW12 Gateron_ks_27, SW13 Gateron_ks_27, SW14 Gateron_ks_27, SW15 Gateron_ks_27, SW16 Gateron_ks_27, SW17 Gateron_ks_27, SW18 Gateron_ks_27, SW19 Gateron_ks_27, SW2 SW_LED_DIODE, SW20 Gateron_ks_27, SW21 Gateron_ks_27, SW22 Gateron_ks_27, SW23 Gateron_ks_27, SW24 Gateron_ks_27, SW25 Gateron_ks_27, SW26 Gateron_ks_27, SW27 Gateron_ks_27, SW28 Gateron_ks_27, SW29 Gateron_ks_27, SW3 SW_LED_DIODE, SW30 Gateron_ks_27, SW31 Gateron_ks_27, SW32 Gateron_ks_27, SW33 Gateron_ks_27, SW34 Gateron_ks_27, SW35 Gateron_ks_27, SW36 Gateron_ks_27, SW37 Gateron_ks_27, SW38 Gateron_ks_27, SW39 Gateron_ks_27, SW4 SW_LED_DIODE, SW40 Gateron_ks_27, SW41 Gateron_ks_27, SW42 Gateron_ks_27, SW43 Gateron_ks_27, SW44 Gateron_ks_27, SW45 Gateron_ks_27, SW46 Gateron_ks_27, SW47 Gateron_ks_27, SW48 Gateron_ks_27, SW49 Gateron_ks_27, SW5 SW_LED_DIODE, SW50 Gateron_ks_27, SW51 Gateron_ks_27, SW52 Gateron_ks_27, SW53 Gateron_ks_27, SW54 Gateron_ks_27, SW55 Gateron_ks_27, SW56 Gateron_ks_27, SW57 Gateron_ks_27, SW58 Gateron_ks_27, SW59 Gateron_ks_27, SW6 Gateron_ks_27, SW60 Gateron_ks_27, SW61 Gateron_ks_27, SW62 SW_LED_DIODE, SW63 SW_LED_DIODE, SW64 SW_LED_DIODE, SW65 SW_LED_DIODE, SW7 Gateron_ks_27, SW8 Gateron_ks_27, SW9 Gateron_ks_27, U1 Arduino_pro_Micro, U2 74HC595, U3 74HC595

Commit message: TMP: fixing RES and RST
Parts:
- moved J1 0.76 mm to (131.3, 29.9)
Connections:
- J1 pad 1: RAW -> GND
- J1 pad 2: GND -> RAW
- J1 pad 5: RST -> ~{RES}
- SW1 pad 2: RST -> ~{RST}
- U1 pad 22: RST -> ~{RST}
- U1 pad 5: unconnected-(U1-Pad5) -> ~{RES}
- U2 pad 10: RST -> Vin
- U3 pad 10: RST -> Vin
Routing:
- net RST: track 155.3 -> 0.00 mm
- net ~{RES}: track 0.00 -> 60.3 mm
- net Vin: track 110.4 -> 143.9 mm
- net ~{RST}: track 0.00 -> 27.5 mm
- net RAW: track 77.1 -> 74.8 mm
Other:
- board text added: "~{RES}"

Commit message: TMP: remove unused stuff
Parts:
- removed D1, D2, D3, D4, D5, D6: LED, Keyboard:LED_D3.0mm
- removed J1: Conn_01x11_Female, Keyboard:PinHeader_01x07
- removed J2: Conn_01x03_Male, Keyboard:PinHeader_01x03
- removed R10, R7, R8, R9: 4K7, Resistor_THT:R_Axial_DIN0207_L6.3mm_D2.5mm_P7.62mm_Horizontal
- removed R5, R6: R_US, Resistor_THT:R_Axial_DIN0207_L6.3mm_D2.5mm_P7.62mm_Horizontal
- removed SW2, SW3, SW4, SW5, SW62, SW63, SW64, SW65: SW_LED_DIODE, Keyboard:SW_LED_ext_DIODE
- moved SW1 26.2 mm to (162.6, 35.6)
- moved U2 19.5 mm to (120.6, 46.1), turned to 83 degrees
- moved U3 17.5 mm to (189.4, 48.3), turned to 97 degrees
- moved R4 16.6 mm to (160.0, 110.5)
- moved R1 15.4 mm to (160.0, 85.1)
- moved R2 15.4 mm to (160.0, 94.0)
- moved R3 15.4 mm to (160.0, 102.9)
- moved SW61 14.1 mm to (304.1, 107.1), turned to 7 degrees
- moved SW9 14.1 mm to (23.5, 107.1), turned to -7 degrees
- moved SW60 13.0 mm to (301.8, 88.2), turned to 7 degrees
- moved SW8 12.9 mm to (25.9, 88.2), turned to -7 degrees
- moved SW57 12.2 mm to (285.2, 109.5), turned to 7 degrees
- moved SW13 12.2 mm to (42.4, 109.5), turned to -7 degrees
- moved SW59 12.2 mm to (299.5, 69.3), turned to 7 degrees
- moved SW7 12.2 mm to (28.2, 69.3), turned to -7 degrees
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Connections:
- R1 pad 2: Net-(D1-Pad2) -> GND
- R2 pad 2: Net-(D2-Pad2) -> GND
- R3 pad 2: Net-(D3-Pad2) -> GND
- R4 pad 2: Net-(D4-Pad2) -> GND
- U1 pad 10: LOCK1 -> unconnected-(U1-Pad10)
- U1 pad 24: RAW -> unconnected-(U1-Pad24)
- U1 pad 5: ~{RES} -> unconnected-(U1-Pad5)
- U1 pad 6: ~{CS} -> unconnected-(U1-Pad6)
- U1 pad 7: D~{C} -> unconnected-(U1-Pad7)
- U1 pad 9: LOCK2 -> unconnected-(U1-Pad9)
- U2 pad 10: Vin -> VCC
- U2 pad 15: COL1 -> unconnected-(U2-Pad15)
- U2 pad 16: Vin -> VCC
- U3 pad 10: Vin -> VCC
- U3 pad 16: Vin -> VCC
- U3 pad 7: COL16 -> unconnected-(U3-Pad7)
Routing:
- net ROW4: track 530.3 -> 215.9 mm
- net ROW3: track 468.6 -> 205.9 mm
- net ROW2: track 449.9 -> 205.8 mm
- net Vin: track 143.9 -> 0.00 mm
- net CLK: track 136.8 -> 0.00 mm
- net ROW1: track 370.9 -> 237.0 mm
- net /left_hand/SPI_OUT: track 97.3 -> 0.00 mm
- net COL2: track 146.2 -> 57.2 mm
- net COL15: track 141.4 -> 57.1 mm
- net COL16: track 83.0 -> 0.00 mm
- net SPI_DATA: track 79.3 -> 0.00 mm
- net RAW: track 74.8 -> 0.00 mm
- net COL1: track 73.2 -> 0.00 mm
- net COL3: track 129.3 -> 57.2 mm
- net COL14: track 125.4 -> 57.1 mm
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Other:
- board size 297.2 x 104.8 mm -> 299.7 x 104.8 mm
- board text removed: "CLK"
- board text removed: "COL1"
- board text removed: "COL16"
- board text removed: "Check"
- board text removed: "DATA"
- board text removed: "D~{C}"
- board text removed: "GND"
- board text removed: "RAW"
- board text removed: "VCC"
- board text removed: "Vin"
- board text removed: "~{CS}"
- board text removed: "~{RES}"
